File: kicad/board3/ProPrj_New Project_2026-07-15_23-14-34_2026-07-27.kicad_sch (KiCad schematic)
At the start: 141 parts, among them P1 WJ500V-5.08-2P, P2 WJ500V-5.08-2P, Q1 AO4406A, Q2 AO4406A, SW1 HX TS4538CJ 250gf 009, SW2 HX TS4538CJ 250gf 009, SW3 HX TS4538CJ 250gf 009, SW4 HX TS4538CJ 250gf 009, SW6 HX TS4538CJ 250gf 009, SW7 HX TS4538CJ 250gf 009, U1 STM32H755ZIT6, U10 ULN2803A, U2 W25Q512JVEIQ TR, U3 TPS563201DDCR, U4 CH224K, U5 LM74700QDBVRQ1, U6 LM74700QDBVRQ1, U7 FM24CL64B-GTR, U8 TJA1051T/3/1J, U9 TJA1051T/3/1J, X1 25MHz

Commit message: fix(kicad): wire BTN1-4 to PC6-PC9, making all four buttons functional
U2. BTN1-BTN4 were single-pin nets terminating at R28.2-R31.2 -- the switch
side and the MCU side were both present and never joined, leaving four dead
buttons on a prototype that wants them.

The fix is four labels, not four wires. KiCad joins nets by label name, and
BTN1-BTN4 labels already existed near the resistors; adding a second label of
the same name at each U1 pin merges the nets with no geometry to get wrong.

Pins chosen for routing, not convenience:

  pad 93  PC6   pad 94  PC7   pad 95  PC8   pad 96  PC9

Four consecutive free pads on U1's west edge, which is the side facing the
button cluster at the board's bottom-left. The south edge faces the CAN
cluster -- both transceivers, termination and jumpers -- so leaving that way
would cross all of it. West runs straight out with nothing in between, and
consecutive pads route as a clean four-wire bus.

They also share one interrupt vector: PC6-PC9 map to EXTI6-EXTI9, and EXTI5-9
share EXTI9_5_IRQn on STM32, so one ISR serves all four buttons. None are
power, VCAP, VREF or boot pins.

One thing to know later: PC8 and PC9 are SDMMC1 D0/D1. Unused today, but an SD
card on this board would collide.

Traces run ~105mm, which is long and fine -- slow signals, internal pull-ups,
switch to ground, and dash_button.h already debounces at 30ms precisely
because EMI on a car harness must not produce a phantom press.

Verified two ways: analyze_schematic.py reports zero NT-001 single-pin nets
(findings 68 -> 64), and the exported netlist shows each /BTN net carrying its
resistor pin plus its U1 pin by name.

The PCB still needs Update PCB from Schematic to pick up the four new
connections as ratlines -- a GUI step.

Co-Authored-By: Claude Opus 5 (1M context) <noreply@anthropic.com>
Connections:
- net BTN1: now also U1.93 (PC6)
- net BTN2: now also U1.94 (PC7)
- net BTN3: now also U1.95 (PC8)
- net BTN4: now also U1.96 (PC9)
Changed lines of the file:
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@@
+	)
+	(label "BTN1"
+		(at 48.26 215.9 0)
+		(effects
+			(font
+				(size 1.2446 1.2446)
+			)
+			(justify left bottom)
+		)
+	)
+	(label "BTN2"
+		(at 48.26 213.36 0)
+		(effects
+			(font
+				(size 1.2446 1.2446)
+			)
+			(justify left bottom)
+		)
+	)
+	(label "BTN3"
+		(at 48.26 210.82 0)
+		(effects
+			(font
+				(size 1.2446 1.2446)
+			)
+			(justify left bottom)
+		)
+	)
+	(label "BTN4"
+		(at 48.26 208.28 0)
+		(effects
+			(font
+				(size 1.2446 1.2446)
+			)
+			(justify left bottom)
+		)
 	)
 	(label "BTN1"

Commit message: chore(kicad): clean schematic residue and re-link board nets (BTN link INCOMPLETE)
Committed as a recoverable checkpoint, not as finished work. One part of this
did not achieve what it was meant to, and the next session needs that stated
plainly rather than inferred from a diff.

Schematic, done:
  * orphaned wire stubs removed (SCLK_C, MOSI_C, MISO_C, CS_C, GND) -- labelled
    segments left behind when a component was deleted in EasyEDA, carried
    across by the import. They named nets that already existed, so they
    contributed no nodes and removing them changed no connectivity.
  * Drawing-Symbol_A4 removed -- EasyEDA's A4 title block, imported as a symbol
    with no designator, value or footprint. It was the phantom BOM line and the
    reason KiCad kept demanding annotation. KiCad draws its own sheet frame.

Board, partially done:
  * Update PCB from Schematic now runs with 0 errors. It previously reported
    one "Cannot add <ref>" per component -- 140 of them -- invariant to every
    option checkbox, because the importer produces a schematic and board whose
    symbol-to-footprint UUID paths do not correspond. The fix is to tick
    "Re-link footprints to schematic symbols based on their reference
    designators", which matches by designator instead. Compounded by the
    importer creating no footprint library at all, so the fallback add path
    could not succeed either.
  * That update reconciled net naming: the board's nets lacked the hierarchical
    "/" prefix the schematic uses, so every via and zone reconnected from GND to
    /GND, +3V3 to /+3V3 and so on.

What did NOT happen, and is the open item:
  * The four BTN1-4 -> U1.93-96 (PC6-PC9) pad assignments did not transfer.
    /BTN1 still carries only R28.2. The schematic is correct and verified --
    the exported netlist shows R28.2 plus U1.93[PC6_93], and analyze_schematic
    reports zero NT-001 single-pin nets -- so this is a transfer failure, not a
    schematic problem. Cause unknown; d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
Parts:
- removed ?: (no value), ProPrj_New-easyedapro:, symbol ProPrj_New-easyedapro:Drawing-Symbol_A4
Connections:
- net BTN1: no longer U1.93 (PC6)
- net BTN2: no longer U1.94 (PC7)
- net BTN3: no longer U1.95 (PC8)
- net BTN4: no longer U1.96 (PC9)

Commit message: fix(kicad): connect BTN1-4 to PC6-PC9, restoring a link that a cleanup deleted
The four buttons were dead because /BTN1-4 never reached the MCU. The prior
session recorded this as a schematic-to-board transfer failure, with the
schematic "correct and verified". It was neither.

git show settles it: 8d7f859 added four labels wiring BTN1-4 to U1.93-96, and
e721f36 deleted exactly those four labels while removing five genuinely
orphaned wire stubs. Its netlist verification ran before its own deletion.

The root cause is the cleanup heuristic. A bare label sitting on a pin has no
wire under it, so "label with no wire endpoint = orphaned residue" removes
working connections. The five stubs it dropped were correct; the four BTN
labels were collateral.

So the fix uses the form the sheet already uses everywhere else: a 2.54 mm
stub (48.26,y)->(50.8,y) with the label at (49.53,y), identical to VBUS_SENSE,
USB_DP, USB_DM, QSPI_NCS, +3V3 and GND on the same pin column. That is not
cosmetic -- the stub is what makes the connection read as intentional to the
next cleanup pass.

Measured, not assumed:
  * netlist: /BTN1=[R28.2,U1.93] /BTN2=[R29.2,U1.94] /BTN3=[R30.2,U1.95]
    /BTN4=[R31.2,U1.96]
  * board: U1 pads 93-96 now carry /BTN1../BTN4; airwires 1 -> 5 (four new
    connections awaiting copper in U5, plus the pre-existing free-pad
    artifact); tracks+vias unchanged at 2557; 144 footprints, none zero-pad
  * ERC delta zero (1265 -> 1265), itemised: -4 isolated_pin_label,
    -4 pin_not_connected, +4 pin_to_pin (imported symbols carry unspecified
    pin types; 317 already existed), +4 unconnected_wire_endpoint (the far end
    of each stub -- the import's own stubs produce 477 of these)

The .kicad_pcb diff is large out of all proportion to the change: consuming
the four unconnected-(U1-PC*-Pad9*) placeholders took net count 221 -> 217 and
KiCad renumbered every net code in the file. Only four pad net assignments are
semantic.

Two things worth carrying forward.

Update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
Connections:
- net BTN1: now also U1.93 (PC6)
- net BTN2: now also U1.94 (PC7)
- net BTN3: now also U1.95 (PC8)
- net BTN4: now also U1.96 (PC9)
Changed lines of the file:
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@@
+	(wire
+		(pts
+			(xy 50.8 215.9) (xy 48.26 215.9)
+		)
+		(stroke
+			(width 0)
+			(type default)
+		)
+	)
+	(wire
+		(pts
+			(xy 50.8 213.36) (xy 48.26 213.36)
+		)
+		(stroke
+			(width 0)
+			(type default)
+		)
+	)
+	(wire
+		(pts
+			(xy 50.8 210.82) (xy 48.26 210.82)
+		)
+		(stroke
+			(width 0)
+			(type default)
+		)
+	)
+	(wire
+		(pts
+			(xy 50.8 208.28) (xy 48.26 208.28)
+		)
+		(stroke
+			(width 0)
+			(type default)
+		)
+	)
 	(wire
 		(pts
@@
 		(effects
 			(font
+				(size 1.2446 1.2446)
+			)
+			(justify left bottom)
+		)
+	)
+	(label "BTN1"
+		(at 49.53 215.9 0)
+		(effects
+			(font
+				(size 1.2446 1.2446)
+			)
+			(justify left bottom)
+		)
+	)
+	(label "BTN2"
+		(at 49.53 213.36 0)
+		(effects
+			(font
+				(size 1.2446 1.2446)
+			)
+			(justify left bottom)
+		)
+	)
+	(label "BTN3"
+		(at 49.53 210.82 0)
+		(effects
+			(font
+				(size 1.2446 1.2446)
+			)
+			(justify left bottom)
+		)
+	)
+	(label "BTN4"
+		(at 49.53 208.28 0)
+		(effects
+			(font

Commit message: feat(kicad): add R49, the 10k NRST pull-up (U3, schematic half)
The STM32H755 has an internal NRST pull-up around 30-50k, so this is EMI margin
rather than a fix -- but the board is going in a car, where a reset line held up
only by an internal pull-up is a line waiting for a transient.

Built by cloning R1, which is already the same part: 0603WAF1002T5E, LCSC C25804,
10k 0603. So no new library symbol, no new footprint association, and no new BOM
line -- the existing 10k row goes from quantity 3 to 4 (R1,R2,R7,R49). That is
also why this was safe to do headlessly: KTD4 calls adding COMPONENTS riskier
than adding connections because of symbol, unit and footprint mapping, and
cloning an identical part sidesteps all three.

Placed at (31.75, 87.63), about 18 mm below C46 in space measured clear by
16.6 mm, wired with 2.54 mm stubs carrying local labels -- the same convention
every other net on this single-sheet schematic uses, and the same one U2's fix
used after a bare label was swept as orphaned residue.

Verified with kicad-cli sch export netlist, which is the netlist KiCad syncs the
board from rather than a proxy for it:

  /NRST  C46.1, H2.4, R49.2, SW6.1, U1.27   (was 4 nodes, now 5)
  /+3V3  74 nodes including R49.1           (was 73)

ERC delta measured with both schematics in the SAME directory, because the first
comparison ran the old one from a scratch path where ${KIPRJMOD} could not
resolve the footprint library and invented a 140-violation improvement. Like for
like it is 1265 -> 1271, +6, all of it one symbol and two stubs: +1 lib_symbol,
+1 footprint_link, +1 pin_not_driven (the +3V3 end), +1 pin_to_pin (imported
symbols carry unspecified pin types; 321 already did) and +2
unconnected_wire_endpoint, one per stub far end -- exactly the signature U2's
four stubs produced, scaled to two.

STILL TO DO, and it is the GUI-only step: Update PCB from Schematic with
"Re-link footprints to schematic symbols based on their reference designators"
ticked. Until the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
Parts:
- added R49: 10kΩ, ProPrj_New-easyedapro:R0603, symbol ProPrj_New-easyedapro:0603WAF1002T5E
Connections:
- net +3V3: now also R49.1
- net NRST: now also R49.2

Commit message: fix(kicad): swap the telltale Darlington for a DMOS array (U10, schematic half)
The ULN2803A's ~0.8 V saturation drop was eating up to 44% of the headroom the
high-Vf telltales need, holding the blue channel to 5 mA. TBD62083AFWG (C165895,
325 mOhm) drops 4.9 mV at 15 mA instead. It also closes a margin nobody chose:
the Darlington's current-driven inputs are specified against 5 V logic and the
H755 drives them at 3.3 V, where the DMOS part is specified for 3 V.

Pin-compatible in the strongest available sense -- both parts resolve to the
same EasyEDA footprint UUID (45c3bbdf...f34), so the Footprint property and the
board file are untouched, and DRC and airwires are unchanged by construction.

The project symbol library is renamed alongside the schematic's cached copy.
Renaming only the cache leaves the .kicad_sym defining a symbol the schematic no
longer references -- a mismatch the netlist check does not catch.

Verified: netlist node-for-node identical (215 nets, 0 added/removed/changed;
U10's 18 pins and all 24 TT nets unchanged); ERC delta 0 (1130 -> 1130 under
matching project config); BOM still 51 lines, 51 sourced, 0 without LCSC or MPN.

Expect brighter telltales until U12. With the 0.8 V handed back to the
resistors, the existing values pass more current -- blue 5.0 -> 9.0 mA, yellow
8.0 -> 10.6 mA, red 9.6 -> 12.6 mA -- all well inside a 20 mA 0805 rating, but
the row stays unmatched until the resistors are re-derived.

Schematic half only: Update PCB from Schematic is GUI-only (KTD12). Restart
KiCad before syncing -- it reads eeschema's cached copy, not the file, and will
otherwise report no changes.

Co-Authored-By: Claude Opus 5 (1M context) <noreply@anthropic.com>
Parts:
- U10: value ULN2803A -> TBD62083AFWG; symbol ProPrj_New-easyedapro:ULN2803A_C181731 -> ProPrj_New-easyedapro:TBD62083AFWG_C165895; Manufacturer Mixic(中科芯亿达) -> TOSHIBA; Manufacturer Part ULN2803A -> TBD62083AFWG; Supplier Part C181731 -> C165895
Changed lines of the file:
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@@
 	)
 	(symbol
-		(lib_id "ProPrj_New-easyedapro:ULN2803A_C181731")
+		(lib_id "ProPrj_New-easyedapro:TBD62083AFWG_C165895")
 		(at 292.1 195.58 0)
 		(unit 1)
@@
 			)
 		)
-		(property "Value" "ULN2803A"
+		(property "Value" "TBD62083AFWG"
 			(at 284.48 210.82 0)
 			(show_name no)
@@
 			)
 		)
-		(property "Datasheet" "https://item.szlcsc.com/datasheet/ULN2803A/193128.html"
+		(property "Datasheet" "https://www.lcsc.com/datasheet/lcsc_datasheet_2304140030_TOSHIBA-TBD62083AFWG-EL_C165895.pdf"
 			(at 292.1 195.58 0)
 			(hide yes)
@@
 			)
 		)
-		(property "Description" "number of channels:8 Collector - Emitter Voltage VCEO:50V Current - Collector(Ic):500mA Voltage - Input(Max):30V Operating Temperature:-40℃~+85℃ Operating Temperature:-40℃~+85℃ Output Leakage Current(Icex):50uA Input Current(on):4mA Voltage - Forward(Vf):"
+		(property "Description" "number of channels:8 RDS(on):325mOhm Voltage - Supply:2.5V~30V Control Input Logic:Active High Operating Temperature:-40C~+85C Type:Low Side Switch"
 			(at 292.1 195.58 0)
 			(hide yes)
@@
 			)
 		)
-		(property "Manufacturer Part" "ULN2803A"
+		(property "Manufacturer Part" "TBD62083AFWG"
 			(at 292.1 195.58 0)
 			(hide yes)
@@
 			)
 		)
-		(property "Manufacturer" "Mixic(中科芯亿达)"
+		(property "Manufacturer" "TOSHIBA"
 			(at 292.1 195.58 0)
 			(hide yes)
@@
 			)
 		)
-		(property "Supplier Part" "C181731"
+		(property "Supplier Part" "C165895"
 			(at 292.1 195.58 0)
 			(hide yes)

Commit message: fix(kicad): correct the telltale annotation, which described a board that never shipped
The note claimed the telltale LEDs and their resistors live off-board on an "H1
telltale header". They do not: LED1-8 and R25/R26/R27/R38/R39/R40/R44/R48 are all
on this board, and H1 is the CAN connector (/CAN1_H, /CAN1_TERM).

Every resistor value in it was fiction too -- it listed 150/82/82/150/180/150/
150/180 against the actual 390/300/200/390/470/270/270/300. Anyone sizing a
telltale from this note would have doubled the current.

Now records the real chain (+5V -> LED -> series resistor -> U10 -> GND), the
verified per-channel LED/resistor/colour/function mapping, the new DMOS driver,
and the H755 rather than the Teensy that has not driven this board in a while.

Text graphic only: no pins, no net, absent from the netlist. Verified inert --
netlist identical but for the export timestamp, ERC unchanged at 1130.

Co-Authored-By: Claude Opus 5 (1M context) <noreply@anthropic.com>
Other:
- note added: "Telltale chain, all on-board: +5V -> LED anode; LED cathode -> series resistor -> U10 output, which sinks to GND when the H755 drives the matching input HIGH. TT1 LED1 GREEN (left turn) R25 390R | TT2 LED3 WHITE (headlight) R27 300R | TT3 LED4 BLUE (high beam) R39 200R | TT4 LED2 GREEN (right turn) R26 390R TT5 LED5 ORANGE (MIL/CEL) R40 470R | TT6 LED6 RED (parking brake) R44 270R | TT7 LED7 RED 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"
- note removed: "H1 telltale header - external LED + series resistor per channel (LEDs/resistors live off-board, wired to dash bezel): Pin1 TT1 = GREEN (left turn) - 150R | Pin2 TT2 = WHITE (headlight) - 82R | Pin3 TT3 = BLUE (high beam) - 82R | Pin4 TT4 = GREEN (right turn) - 150R Pin5 TT5 = ORANGE (MIL/CEL) - 180R | Pin6 TT6 = RED (parking brake) - 150R | Pin7 TT7 = RED (oil pressure) - 150R | Pin8 TT8 = YELLOW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"
Changed lines of the file:
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@@
 		)
 	)
-	(text "H1 telltale header - external LED + series resistor per channel (LEDs/resistors live off-board, wired to dash bezel):\nPin1 TT1 = GREEN (left turn) - 150R | Pin2 TT2 = WHITE (headlight) - 82R | Pin3 TT3 = BLUE (high beam) - 82R | Pin4 TT4 = GREEN (right turn) - 150R\nPin5 TT5 = ORANGE (MIL/CEL) - 180R | Pin6 TT6 = RED (parking brake) - 150R | Pin7 TT7 = RED (oil pressure) - 150R | Pin8 TT8 = YELLOW (fog lights) - 180R\nPin9 = +5V (LED anode supply, common) | Pin10 = GND\nWiring per LED: +5V -> series resistor (value above) -> LED anode; LED cathode -> this pin (ULN2803A sinks to GND when Teensy pin HIGH)."
+	(text "Telltale chain, all on-board: +5V -> LED anode; LED cathode -> series resistor -> U10 output, which sinks to GND when the H755 drives the matching input HIGH.\nTT1 LED1 GREEN (left turn) R25 390R | TT2 LED3 WHITE (headlight) R27 300R | TT3 LED4 BLUE (high beam) R39 200R | TT4 LED2 GREEN (right turn) R26 390R\nTT5 LED5 ORANGE (MIL/CEL) R40 470R | TT6 LED6 RED (parking brake) R44 270R | TT7 LED7 RED (oil pressure) R48 270R | TT8 LED8 YELLOW (fog lights) R38 300R\nDriver U10 = TBD62083AFWG DMOS array, ~5 mV on-state drop. The resistor values above predate that swap and are still to be re-derived for it; until then the row runs brighter and unmatched."
 		(exclude_from_sim no)
 		(at 222.25 249.174 0)
