File: kicad/board3/ProPrj_New Project_2026-07-15_23-14-34_2026-07-27.kicad_sch (KiCad schematic)
At the start: 141 parts, among them P1 WJ500V-5.08-2P, P2 WJ500V-5.08-2P, Q1 AO4406A, Q2 AO4406A, SW1 HX TS4538CJ 250gf 009, SW2 HX TS4538CJ 250gf 009, SW3 HX TS4538CJ 250gf 009, SW4 HX TS4538CJ 250gf 009, SW6 HX TS4538CJ 250gf 009, SW7 HX TS4538CJ 250gf 009, U1 STM32H755ZIT6, U10 TBD62083AFWG, U2 W25Q512JVEIQ TR, U3 TPS563201DDCR, U4 CH224K, U5 LM74700QDBVRQ1, U6 LM74700QDBVRQ1, U7 FM24CL64B-GTR, U8 TJA1051T/3/1J, U9 TJA1051T/3/1J, X1 25MHz

Commit message: feat(kicad): move the eight telltales to 3528, polarity normalised (U11)
LED1-8 leave the 0805 generics for the HONGLITRONIC 3528 set chosen in
KTD13, and every position is now wired pin 1 = cathode, pin 2 = anode. The
board previously split 4/4 between the two conventions because the six
imported symbols disagreed with each other.

Two geometry compensations were needed and neither is obvious from the
diff:

The replacements put their pins at library y=0; the parts they replace did
not. KiCad negates library y onto the canvas, so LED1 and LED2 shift +1.016
and LED3 shifts +1.270 to keep the existing wires landing on the pins. Skip
this and the wires silently detach.

The red HL-A-3528S35FC is mirrored against its five siblings -- anode at
library x -5.08 where every other part, old and new, puts it at +5.08 -- so
LED6 and LED7 take (mirror y). Skip this and those two telltales are fitted
backwards, which no gate would catch: netlist, ERC, DRC and the BOM all pass
a reversed LED, and it shows up only as a dead indicator at bring-up.

Verified by netlist export rather than inspection: all sixteen nodes land
correctly, every pin 2 on /+5V carrying A or +, every pin 1 on its
/TT*_LED_K carrying C, K or -, and each telltale keeps its original net
(LED2 to TT4, LED3 to TT2, and so on).

ERC 171 violations, identical to the pre-change baseline -- zero delta.
kicad_lcsc check PASS 141/141 mapped and modelled; duplicates exit 0 with
50 distinct codes, six out and six in.

The board still carries 0805 land patterns until Update PCB from Schematic
runs in the GUI, so it is deliberately not fab-ready at this commit.

Co-Authored-By: Claude Opus 5 (1M context) <noreply@anthropic.com>
Parts:
- LED1, LED2: value NCD0805G1 -> HL-A-3528U51GC-S1-13HL; footprint ProPrj_New-easyedapro:LED0805-R-RD -> JLCImport:HL-A-3528U51GC-S1-13HL; symbol ProPrj_New-easyedapro:FC-2012UGK-520D5 -> JLCImport:HL-A-3528U51GC-S1-13HL; Illumination Color Green -> Emerald Green; LCSC Part Name 片式发光二极管 -> HL-A-3528U51GC-S1-13HL; Lens Color - -> Water Clear; Luminous Intensity 400mcd -> 1.3cd; Manufacturer 国星光电 -> HONGLITRONIC(Hongli Zhihui (HONGLITRONIC)); Manufacturer Part NCD0805G1 -> HL-A-3528U51GC-S1-13HL; Operating Temperature -30℃~+85℃ -> -40℃~+85℃; Peak Wavelength 520nm -> -; Power(Watts) 72mW -> 102mW; Supplier Part C84260 -> C516142; Viewing Angle 130° -> 120°; Voltage - Forward(Vf) 2.5V~3.6V -> 3.4V; Wavelength - Dominant 525nm~537.5nm -> 515nm~525nm
- LED3: value KT-0805W -> HL-A-3528H343W-S1-13HL-HR3_SDCM_amp_lt_6_6000K-7000K; footprint ProPrj_New-easyedapro:LED0805-R-RD -> JLCImport:HL-A-3528H343W-S1-13HL-HR3_SDCM_amp_lt_6_6000K-7000K; symbol ProPrj_New-easyedapro:whiteLEDSMD -> JLCImport:HL-A-3528H343W-S1-13HL-HR3_SDCM_amp_lt_6_6000K-7000K; Color Temperature 13172K~100000K -> 6500K; Forward Current 25mA -> 20mA; JLCPCB Part Class Basic Part -> Extended Part; LCSC Part Name 0805 白灯 高亮 -> HL-A-3528H343W-S1-13HL-HR3_SDCM_amp_lt_6_6000K-7000K; Lens Color Yellow Lens -> Frosted Yellow Lens; Luminous Intensity 350mcd -> -; Manufacturer KENTO -> HONGLITRONIC(Hongli Zhihui (HONGLITRONIC)); Manufacturer Part KT-0805W -> HL-A-3528H343W-S1-13HL-HR3_SDCM_amp_lt_6_6000K-7000K; Operating Temperature -30℃~+85℃ -> -40℃~+85℃; Power(Watts) 80mW -> 96mW; Supplier Part C34499 -> C516299; Voltage - Forward(Vf) 2.6V~3.2V -> 3.2V
- LED4: value XL-2012UBC -> HL-A-3528H203BC-S1-13HL; footprint ProPrj_New-easyedapro:LED0805-RD -> JLCImport:HL-A-3528H203BC-S1-13HL; symbol ProPrj_New-easyedapro:XL-2012UBC -> JLCImport:HL-A-3528H203BC-S1-13HL; LCSC Part Name 0805蓝贴片式发光二极管 -> HL-A-3528H203BC-S1-13HL; Luminous Intensity 260mcd -> 350mcd; Manufacturer XINGLIGHT(成兴光) -> HONGLITRONIC(Hongli Zhihui (HONGLITRONIC)); Manufacturer Part XL-2012UBC -> HL-A-3528H203BC-S1-13HL; Peak Wavelength 470nm -> -; Power(Watts) 70mW -> 102mW; Supplier Part C965817 -> C516143; Voltage - Forward(Vf) 3.2V -> 3.4V; Wavelength - Dominant 460nm~475nm -> 464nm~474nm
- LED5: value XL-2012UOC -> HVO-3528CPXA; footprint ProPrj_New-easyedapro:LED0805-RD_ORANGE -> JLCImport:HVO-3528CPXA; symbol ProPrj_New-easyedapro:XL-2012UOC -> JLCImport:HVO-3528CPXA; LCSC Part Name 0805橙贴片式发光二极管 -> HVO-3528CPXA; Lens Color Water Clear -> White Lens; Luminous Intensity 330mcd -> 1.8cd; Manufacturer XINGLIGHT(成兴光) -> HONGLITRONIC(Hongli Zhihui (HONGLITRONIC)); Manufacturer Part XL-2012UOC -> HVO-3528CPXA; Operating Temperature -40℃~+85℃ -> -40℃~+100℃; Peak Wavelength 605nm -> 610nm; Power(Watts) 50mW -> -; Supplier Part C965813 -> C5246349; Voltage - Forward(Vf) 2.3V -> 2.2V; Wavelength - Dominant 600nm~610nm -> 600nm~609nm
- LED6, LED7: value NCD0805R1 -> HL-A-3528S35FC-S1-13HL; footprint ProPrj_New-easyedapro:LED0805-RD -> JLCImport:HL-A-3528S35FC-S1-13HL; symbol ProPrj_New-easyedapro:FC-2012HRK-620D -> JLCImport:HL-A-3528S35FC-S1-13HL; Forward Current 25mA -> 20mA; JLCPCB Part Class Basic Part -> Extended Part; LCSC Part Name 片式发光二极管 -> HL-A-3528S35FC-S1-13HL; Lens Color - -> Water Clear; Luminous Intensity 195mcd -> 270mcd; Manufacturer 国星光电 -> HONGLITRONIC(Hongli Zhihui (HONGLITRONIC)); Manufacturer Part NCD0805R1 -> HL-A-3528S35FC-S1-13HL; Operating Temperature -30℃~+85℃ -> -40℃~+85℃; Peak Wavelength 630nm -> -; Power(Watts) 65mW -> 72mW; Supplier Part C84256 -> C516141; Viewing Angle 130° -> 120°; Voltage - Forward(Vf) 1.6V~2.6V -> 2.4V; Wavelength - Dominant 615nm~630nm -> 617nm~627nm
- LED8: value KT-0805Y -> HL-A-3528S31YC-S1-13HL; footprint ProPrj_New-easyedapro:LED0805-R-RD -> JLCImport:HL-A-3528S31YC-S1-13HL; symbol ProPrj_New-easyedapro:17-21SUYC/TR8 -> JLCImport:HL-A-3528S31YC-S1-13HL; Forward Current - -> 20mA; JLCPCB Part Class Basic Part -> Extended Part; LCSC Part Name 0805 黄灯 高亮 -> HL-A-3528S31YC-S1-13HL; Luminous Intensity 175mcd -> 210mcd; Manufacturer KENTO -> HONGLITRONIC(Hongli Zhihui (HONGLITRONIC)); Manufacturer Part KT-0805Y -> HL-A-3528S31YC-S1-13HL; Peak Wavelength 596nm -> -; Power(Watts) 40mW -> 72mW; Supplier Part C2296 -> C516140; Voltage - Forward(Vf) 1.8V~2.4V -> 2.4V; Wavelength - Dominant 584nm~594nm -> 583nm~593nm
Connections:
- net +5V: now also LED1.2 (A), LED2.2 (A), LED3.2 (A), LED8.2 (+); no longer LED1.1 (A), LED2.1 (A), LED3.1 (A), LED8.1 (+)
- net TT1_LED_K: now also LED1.1 (C); no longer LED1.2 (K)
- net TT2_LED_K: now also LED3.1 (C); no longer LED3.2 (K)
- net TT4_LED_K: now also LED2.1 (C); no longer LED2.2 (K)
- net TT8_LED_K: now also LED8.1 (-); no longer LED8.2 (-)

Commit message: feat(kicad): CS_R to PE3, PD_R off the +5V plane (U18)
The two pin-assignment artifacts the U1 placement review found are fixed.
DRC NEW = 0 against the pre-change board, unconnected 0, exactly two nets
changed (CS_R, PD_R), via-in-pad audit unchanged, ERC 171 with zero delta,
netlist diff exactly /CS_R -[U1,78] +[U1,2].

CS_R moves from PD10 (pin 78, west edge) to PE3 (pin 2, east edge) -- a free
full-speed GPIO sitting in the middle of the right-panel SPI escape group.
The net no longer crosses the entire package to reach FPC3: it escapes east,
rides the empty bottom layer at y=118.9, and rejoins its own tail at the
vacated y=103.496 lane. Carrier firmware note: right-panel chip select is
PE3 (the firmware does not exist yet, so this is a #define, not a port).

PD_R keeps its pin -- its defect was the route, not the assignment. It ran
71 mm through Inner2, cutting the +5V plane diagonally through the crystal
region and along y=93.5. It now inherits CS_R's vacated corridor (bottom
y=103.496 plus the top lane) and reaches its FPC3 tail by diving under the
+5V wall at the connector and resurfacing through the OLD via at
(222.842,93.532), kept because a through-via serves the bottom layer as well
as it served Inner2. The +5V plane under the right-panel bus is whole again.

Why PD_R did not also get a new pin: the PE3/PE4 escape pocket is fenced by
a GND corner stitch and already holds the three SPI_R vias -- exhaustive
placement showed it fits exactly one more via. The north-edge free pins
(PA0/PA4) are walled in by a +3V3 L-shape and a GND diagonal.

Residual, stated plainly: the y=103.496 bottom crossing under the crystal
corner still exists -- it belongs to PD_R now -- so plan 002's note that
QSPI_CLK carries 4 vias to cross it still stands.

Three revisions to land it, each driven by a measured failure: the join via
could not sit on the tail start (a GND diagonal parallels the tail at 0.494,
legal for the track, illegal for a via); the retreat position sat 0.226 f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
Connections:
- net CS_R: now also U1.2 (PE3); no longer U1.78 (PD10)
Changed lines of the file:
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@@
 	(wire
 		(pts
-			(xy 50.8 254) (xy 48.26 254)
+			(xy 1.27 88.9) (xy 2.54 88.9)
 		)
 		(stroke
@@
 	)
 	(label "CS_R"
-		(at 49.53 254 0)
+		(at 1.27 88.9 180)
 		(effects
 			(font
 				(size 1.2446 1.2446)
 			)
-			(justify left bottom)
+			(justify right bottom)
 		)
 	)
