File: kicad/board3/ProPrj_New Project_2026-07-15_23-14-34_2026-07-27.kicad_sch (KiCad schematic)
At the start: 141 parts, among them P1 WJ500V-5.08-2P, P2 WJ500V-5.08-2P, Q1 AO4406A, Q2 AO4406A, SW1 HX TS4538CJ 250gf 009, SW2 HX TS4538CJ 250gf 009, SW3 HX TS4538CJ 250gf 009, SW4 HX TS4538CJ 250gf 009, SW6 HX TS4538CJ 250gf 009, SW7 HX TS4538CJ 250gf 009, U1 STM32H755ZIT6, U11 AW9523BTQR, U12 AW9523BTQR, U2 W25Q256JVEIQ, U3 TPS563201DDCR, U4 CH224K, U5 LM74700QDBVRQ1, U6 LM74700QDBVRQ1, U7 FM24CL64B-GTR, U8 TJA1051T/3/1J, U9 TJA1051T/3/1J, X1 25MHz

Commit message: fix(kicad): U54 -- SW1-SW4 were on the wrong land pattern, and would not have fitted
Review item 37, which the review filed under "simplification" as "one part on
two land patterns". It is a fit defect.

All six buttons are C5340169 (hanxia HX TS4538CJ), but SW1-SW4 sat on
SW-TH_4P-...-LS5.4 (pads +/-2.700) and SW6/SW7 on LS5.0 (pads +/-2.500). Both
agree on the 3.00 mm row pitch and both drill 1.0 mm; they disagree by 0.4 mm
of lead span, and the part has one true span.

Settled from the vendor drawing: the recommended PCB pattern is 5 mm x 3 mm,
holes dia 1. LS5.0 is correct and SW6/SW7 were right all along. Reading it
needed a rasteriser -- the drawing is vector, the only embedded image is the
vendor logo, and the callouts do not survive text extraction.

This is not a margin. The same drawing gives the leads as 4-dia 0.95 +/-0.1
into dia 1.0 holes: 0.025 mm of radial slack at nominal and none at the +0.1
lead tolerance. Nothing absorbs 0.2 mm per side, so SW1-SW4 would not have
seated without splaying the leads. An earlier note in the triage doc guessed
"probably still seats" from an assumed 0.5-0.6 mm lead; that was wrong by 2x.

Root cause: SW1-SW4 were placed from a different library symbol -- 4.5X4.5X4.5
WATERPROOF TACT SWITCH DIP 260G, whose 5.4 mm pattern is presumably right for
that part -- and the value and supplier fields were later overridden to the
TS4538CJ without the footprint following.

Fixed on both sides. The board footprints are swapped preserving position,
rotation, reference, value and attributes, with every pad's net carried across
BY PAD NUMBER; the schematic's Footprint field is updated to match, because
--schematic-parity is the only check that compares a footprint to its symbol
and a board-only edit would have left them disagreeing.

Three things came free:
- BOM 42 -> 41 lines. The same LCSC part was ordered as two lines (4 + 2)
  purely because of the footprint split. kicad_lcsc.py duplicates had been
  hinting at this with "41 distinc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
Parts:
- SW1, SW2, SW3, SW4: footprint ProPrj_New-easyedapro:SW-TH_4P-L4.5-W4.5-P3.00-LS5.4 -> ProPrj_New-easyedapro:SW-TH_4P-L4.5-W4.5-P3.00-LS5.0
- SW6, SW7: Manufacturer hanxia(韩下) -> hanxia
Changed lines of the file:
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@@
 			)
 		)
-		(property "Footprint" "ProPrj_New-easyedapro:SW-TH_4P-L4.5-W4.5-P3.00-LS5.4"
+		(property "Footprint" "ProPrj_New-easyedapro:SW-TH_4P-L4.5-W4.5-P3.00-LS5.0"
 			(at 425.45 256.54 0)
 			(hide yes)
@@
 			)
 		)
-		(property "Footprint" "ProPrj_New-easyedapro:SW-TH_4P-L4.5-W4.5-P3.00-LS5.4"
+		(property "Footprint" "ProPrj_New-easyedapro:SW-TH_4P-L4.5-W4.5-P3.00-LS5.0"
 			(at 374.65 256.54 0)
 			(hide yes)
@@
 			)
 		)
-		(property "Footprint" "ProPrj_New-easyedapro:SW-TH_4P-L4.5-W4.5-P3.00-LS5.4"
+		(property "Footprint" "ProPrj_New-easyedapro:SW-TH_4P-L4.5-W4.5-P3.00-LS5.0"
 			(at 450.85 256.54 0)
 			(hide yes)
@@
 			)
 		)
-		(property "Footprint" "ProPrj_New-easyedapro:SW-TH_4P-L4.5-W4.5-P3.00-LS5.4"
+		(property "Footprint" "ProPrj_New-easyedapro:SW-TH_4P-L4.5-W4.5-P3.00-LS5.0"
 			(at 400.05 256.54 0)
 			(hide yes)
@@
 			)
 		)
-		(property "Manufacturer" "hanxia(韩下)"
+		(property "Manufacturer" "hanxia"
 			(at 382.27 274.32 0)
 			(hide yes)
@@
 			)
 		)
-		(property "Manufacturer" "hanxia(韩下)"
+		(property "Manufacturer" "hanxia"
 			(at 408.94 274.32 0)
 			(hide yes)

Commit message: fix(fab): C41/C42 move to a Basic 18pF, dropping an Extended BOM line
Review item 36. The crystal load caps were C527046 (YAGEO CC0603FRNPO9BN180,
18pF +/-1% NP0 0603, Extended). They are now C1647 -- Samsung CL10C180JB8NNNC,
18pF 50V C0G +/-5% 0603, Basic, 524k in stock at $0.0109. Extended BOM lines
26 -> 25.

Identical value, footprint and nets, so the board is untouched and there is no
GUI sync.

The tolerance relaxation is the only real question, and it clears by 45x.
Going +/-1% to +/-5% on an 18pF pair moves the effective crystal load by
+/-0.45 pF around CL = 12 pF. For a 25 MHz fundamental with C0 ~ 3 pF and
C1 ~ 5 fF that is about +/-5 ppm of pull, against +/-1 ppm for the +/-1% part,
so the total budget goes from roughly +/-30 ppm (crystal +/-10 initial, +/-20
over temperature) to +/-35. The tightest consumer here is CAN bit timing at
roughly +/-1580 ppm, and USB does not depend on HSE at all -- DFU runs
HSI48+CRS per AN2606 section 52. The +/-1% part was over-specified.

kicad_lcsc.py add C1647 brought the part in properly, with symbol, footprint
and STEP model in the JLCImport library, and the two instances' supplier
fields were repointed to it.

One deliberate loose end, recorded rather than hidden: C41/C42 still carry
lib_id ProPrj_New-easyedapro:CC0603FRNPO9BN180 and only their instance fields
name the Samsung part. Fully repointing lib_id means hand-inserting a symbol
definition into the schematic's 60k-line lib_symbols cache -- s-expression
surgery for no functional gain, since the BOM is generated from instance
properties and is correct. The on-disk library symbol was left describing the
YAGEO part, because that is what it is. The canonical tidy-up is a GUI Change
Symbol whenever the project is next open. The board already relies on this
same instance-override pattern for SW1-SW4.

Verified: DRC 0 violations / 0 unconnected / 0 schematic parity, ERC unchanged
at 1127, lcsc check passes, duplicates 41 codes and 41 keys, BOM 41 / CPL 140
symmetric.
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
Parts:
- C41, C42: JLCPCB Part Class Extended Part -> Basic Part; LCSC Part Name 18pF ±1% 50V -> 18pF ±5% 50V; Manufacturer YAGEO(国巨) -> Samsung Electro-Mechanics; Manufacturer Part CC0603FRNPO9BN180 -> CL10C180JB8NNNC; Supplier Part C527046 -> C1647
Changed lines of the file:
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@@
 			)
 		)
-		(property "Datasheet" "https://item.szlcsc.com/datasheet/CC0603FRNPO9BN180/545472.html"
+		(property "Datasheet" "https://www.lcsc.com/datasheet/lcsc_datasheet_2304140030_Samsung-Electro-Mechanics-CL10C180JB8NNNC_C1647.pdf"
 			(at 97.79 21.59 0)
 			(hide yes)
@@
 			)
 		)
-		(property "Description" "Capacitance:18pF Tolerance:±1% Tolerance:±1% Voltage Rating:50V Temperature Coefficient:NP0"
+		(property "Description" "Capacitance:18pF Tolerance:±5% Voltage Rating:50V Temperature Coefficient:C0G Package:0603"
 			(at 97.79 21.59 0)
 			(hide yes)
@@
 			)
 		)
-		(property "Manufacturer Part" "CC0603FRNPO9BN180"
+		(property "Manufacturer Part" "CL10C180JB8NNNC"
 			(at 97.79 21.59 0)
 			(hide yes)
@@
 			)
 		)
-		(property "Manufacturer" "YAGEO(国巨)"
+		(property "Manufacturer" "Samsung Electro-Mechanics"
 			(at 97.79 21.59 0)
 			(hide yes)
@@
 			)
 		)
-		(property "Supplier Part" "C527046"
+		(property "Supplier Part" "C1647"
 			(at 97.79 21.59 0)
 			(hide yes)
@@
 			)
 		)
-		(property "LCSC Part Name" "18pF ±1% 50V"
+		(property "LCSC Part Name" "18pF ±5% 50V"
 			(at 97.79 21.59 0)
 			(hide yes)
@@
 			)
 		)
-		(property "JLCPCB Part Class" "Extended Part"
+		(property "JLCPCB Part Class" "Basic Part"
 			(at 97.79 21.59 0)
 			(hide yes)
@@
 			)
 		)
-		(property "Datasheet" "https://item.szlcsc.com/datasheet/CC0603FRNPO9BN180/545472.html"
+		(property "Datasheet" "https://www.lcsc.com/datasheet/lcsc_datasheet_2304140030_Samsung-Electro-Mechanics-CL10C180JB8NNNC_C1647.pdf"
 			(at 113.03 19.05 0)
 			(hide yes)
@@
 			)
 		)
-		(property "Description" "Capacitance:18pF Tolerance:±1% Tolerance:±1% Voltage Rating:50V Temperature Coefficient:NP0"
+		(property "Description" "Capacitance:18pF Tolerance:±5% Voltage Rating:50V Temperature Coefficient:C0G Package:0603"
 			(at 113.03 19.05 0)
 			(hide yes)
@@
 			)
 		)
-		(property "Manufacturer Part" "CC0603FRNPO9BN180"
+		(property "Manufacturer Part" "CL10C180JB8NNNC"
 			(at 113.03 19.05 0)
 			(hide yes)
@@
 			)
 		)
-		(property "Manufacturer" "YAGEO(国巨)"
+		(property "Manufacturer" "Samsung Electro-Mechanics"
 			(at 113.03 19.05 0)
 			(hide yes)
@@
 			)
 		)
-		(property "Supplier Part" "C527046"
+		(property "Supplier Part" "C1647"
 			(at 113.03 19.05 0)
 			(hide yes)
@@
 			)
 		)
-		(property "LCSC Part Name" "18pF ±1% 50V"
+		(property "LCSC Part Name" "18pF ±5% 50V"
 			(at 113.03 19.05 0)
 			(hide yes)
@@
 			)
 		)
-		(property "JLCPCB Part Class" "Extended Part"
+		(property "JLCPCB Part Class" "Basic Part"
 			(at 113.03 19.05 0)
 			(hide yes)

Commit message: fix(kicad): U57 -- CAN termination gets a 500 mW part, and /CAN2_TX moves aside
Review item 17. All four termination resistors (R10/R14/R15/R24, 60.4 ohm)
were 0603/100 mW. A CANH-to-12 V short -- the canonical automotive CAN failure
-- drives 78-87 mA through the series pair at a realistic CANL, so 0.37-0.46 W
each, 3.7-4.6x rating. Only live with the H1/H3 jumper fitted, and not a
functional defect today (thick film fails open, so the bus just loses
termination), but the board is going in a car.

All four go to C3959530, Panasonic ERJP06F60R4V, 0805, 500 mW, 400 V
anti-surge. The part matters more than the size: a common 0805 is 125 mW and
an uprated one 250 mW, both still over.

THE 1206 (660 mW) WAS TRIED FIRST AND REJECTED ON MEASUREMENT. It does not
fit -- R10 fouled R14, R24 fouled P2, and R15 cannot be a vertical 1206 at all
(it needs 5.116 mm between /CAN2_RX and /CAN2_TX and there are 4.246), so it
must rotate and move 2.5 mm east, dragging /CAN2_TERM across /CAN2_TX. Every
arrangement ended in a three-net re-layout, to buy margin on a fault that
needs two simultaneous harness shorts.

R24 STILL HAD NO LEGAL POSITION even as an 0805: a 168-point 2D sweep found
nothing better than +0.051 mm against a 0.1016 mm rule. It is pinned --
/CAN2_L must run west at y=130 to P2.2 and P2 blocks any further west -- and
the /CAN2_TX dogleg cannot move either, because west of x~132 TX must stay
above /CAN2_L and below /CAN2_RX while east of x~134 it is at y=131.579, so
the step is forced into exactly R24's pocket.

So the dogleg drops to the Bottom layer: three segments re-laid identically
with a via at each end, /CAN2_TX length unchanged at 44.459 mm. Bottom in that
pocket was empty, and /CAN2_RX already layer-hops through the same corner on
Inner2. After that R24 does not move at all, and neither do R10, R14 or their
tracks -- only R15 shifts 0.70 mm north.

Both candidate footprints arrived from JLCImport with no courtyard; one was
authored at a 0.25 mm pad margin bef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
Parts:
- R10, R14, R15, R24: footprint ProPrj_New-easyedapro:R0603 -> JLCImport:ERJP06F60R4V; LCSC Part Name 60.4Ω ±1% 100mW 厚膜电阻 -> ERJP06F60R4V; Manufacturer FOJAN(富捷) -> PANASONIC; Manufacturer Part FRC0603F60R4TS -> ERJP06F60R4V; Supplier Part C2933247 -> C3959530
Changed lines of the file:
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@@
 			)
 		)
-		(property "Footprint" "ProPrj_New-easyedapro:R0603"
+		(property "Footprint" "JLCImport:ERJP06F60R4V"
 			(at 120.65 187.96 0)
 			(hide yes)
@@
 			)
 		)
-		(property "Datasheet" "https://item.szlcsc.com/datasheet/FRC0603F60R4TS/3279349.html"
+		(property "Datasheet" "https://item.szlcsc.com/142685.html"
 			(at 120.65 187.96 0)
 			(hide yes)
@@
 			)
 		)
-		(property "Description" "Type:Thick Film Resistor Resistance:60.4Ω Tolerance:±1% Tolerance:±1% Power(Watts):100mW Voltage-Supply(Max):75V Temperature Coefficient:±100ppm/℃ Temperature Coefficient:±100ppm/℃ Operating Temperature:-55℃~+155℃ Operating Temperature:-55℃~+155℃"
+		(property "Description" "Type:Thick Film Resistor Resistance:60.4Ω Tolerance:±1% Power(Watts):500mW Voltage-Supply(Max):400V Temperature Coefficient:±100ppm/℃ Operating Temperature:-55℃~+155℃"
 			(at 120.65 187.96 0)
 			(hide yes)
@@
 			)
 		)
-		(property "Manufacturer Part" "FRC0603F60R4TS"
+		(property "Manufacturer Part" "ERJP06F60R4V"
 			(at 120.65 187.96 0)
 			(hide yes)
@@
 			)
 		)
-		(property "Manufacturer" "FOJAN(富捷)"
+		(property "Manufacturer" "PANASONIC"
 			(at 120.65 187.96 0)
 			(hide yes)
@@
 			)
 		)
-		(property "Supplier Part" "C2933247"
+		(property "Supplier Part" "C3959530"
 			(at 120.65 187.96 0)
 			(hide yes)
@@
 			)
 		)
-		(property "LCSC Part Name" "60.4Ω ±1% 100mW 厚膜电阻"
+		(property "LCSC Part Name" "ERJP06F60R4V"
 			(at 120.65 187.96 0)
 			(hide yes)
@@
 			)
 		)
-		(property "Footprint" "ProPrj_New-easyedapro:R0603"
+		(property "Footprint" "JLCImport:ERJP06F60R4V"
 			(at 91.44 199.39 0)
 			(hide yes)
@@
 			)
 		)
-		(property "Datasheet" "https://item.szlcsc.com/datasheet/FRC0603F60R4TS/3279349.html"
+		(property "Datasheet" "https://item.szlcsc.com/142685.html"
 			(at 91.44 199.39 0)
 			(hide yes)
@@
 			)
 		)
-		(property "Description" "Type:Thick Film Resistor Resistance:60.4Ω Tolerance:±1% Tolerance:±1% Power(Watts):100mW Voltage-Supply(Max):75V Temperature Coefficient:±100ppm/℃ Temperature Coefficient:±100ppm/℃ Operating Temperature:-55℃~+155℃ Operating Temperature:-55℃~+155℃"
+		(property "Description" "Type:Thick Film Resistor Resistance:60.4Ω Tolerance:±1% Power(Watts):500mW Voltage-Supply(Max):400V Temperature Coefficient:±100ppm/℃ Operating Temperature:-55℃~+155℃"
 			(at 91.44 199.39 0)
 			(hide yes)
@@
 			)
 		)
-		(property "Manufacturer Part" "FRC0603F60R4TS"
+		(property "Manufacturer Part" "ERJP06F60R4V"
 			(at 91.44 199.39 0)
 			(hide yes)
@@
 			)
 		)
-		(property "Manufacturer" "FOJAN(富捷)"
+		(property "Manufacturer" "PANASONIC"
 			(at 91.44 199.39 0)
 			(hide yes)
@@
 			)
 		)
-		(property "Supplier Part" "C2933247"
+		(property "Supplier Part" "C3959530"
 			(at 91.44 199.39 0)
 			(hide yes)
@@
 			)
 		)
-		(property "LCSC Part Name" "60.4Ω ±1% 100mW 厚膜电阻"
+		(property "LCSC Part Name" "ERJP06F60R4V"
 			(at 91.44 199.39 0)
 			(hide yes)
@@
 			)
 		)
-		(property "Footprint" "ProPrj_New-easyedapro:R0603"
+		(property "Footprint" "JLCImport:ERJP06F60R4V"
 			(at 106.68 199.39 0)
 			(hide yes)
@@
 			)
 		)
-		(property "Datasheet" "https://item.szlcsc.com/datasheet/FRC0603F60R4TS/3279349.html"
+		(property "Datasheet" "https://item.szlcsc.com/142685.html"
 			(at 106.68 199.39 0)
 			(hide yes)
@@
 			)
 		)
-		(property "Description" "Type:Thick Film Resistor Resistance:60.4Ω Tolerance:±1% Tolerance:±1% Power(Watts):100mW Voltage-Supply(Max):75V Temperature Coefficient:±100ppm/℃ Temperature Coefficient:±100ppm/℃ Operating Temperature:-55℃~+155℃ Operating Temperature:-55℃~+155℃"
+		(property "Description" "Type:Thick Film Resistor Resistance:60.4Ω Tolerance:±1% Power(Watts):500mW Voltage-Supply(Max):400V Temperature Coefficient:±100ppm/℃ Operating Temperature:-55℃~+155℃"
 			(at 106.68 199.39 0)
 			(hide yes)
@@
 			)
 		)
-		(property "Manufacturer Part" "FRC0603F60R4TS"
+		(property "Manufacturer Part" "ERJP06F60R4V"
 			(at 106.68 199.39 0)
 			(hide yes)
@@
 			)
 		)
-		(property "Manufacturer" "FOJAN(富捷)"
+		(property "Manufacturer" "PANASONIC"
 			(at 106.68 199.39 0)
 			(hide yes)
@@
 			)
 		)
-		(property "Supplier Part" "C2933247"
+		(property "Supplier Part" "C3959530"
 			(at 106.68 199.39 0)
 			(hide yes)
@@
 			)
 		)
-		(property "LCSC Part Name" "60.4Ω ±1% 100mW 厚膜电阻"
+		(property "LCSC Part Name" "ERJP06F60R4V"
 			(at 106.68 199.39 0)
 			(hide yes)
@@
 			)
 		)
-		(property "Footprint" "ProPrj_New-easyedapro:R0603"
+		(property "Footprint" "JLCImport:ERJP06F60R4V"
 			(at 134.62 199.39 0)
 			(hide yes)
@@
 			)
 		)
-		(property "Datasheet" "https://item.szlcsc.com/datasheet/FRC0603F60R4TS/3279349.html"
+		(property "Datasheet" "https://item.szlcsc.com/142685.html"
 			(at 134.62 199.39 0)
 			(hide yes)
@@
 			)
 		)
-		(property "Description" "Type:Thick Film Resistor Resistance:60.4Ω Tolerance:±1% Tolerance:±1% Power(Watts):100mW Voltage-Supply(Max):75V Temperature Coefficient:±100ppm/℃ Temperature Coefficient:±100ppm/℃ Operating Temperature:-55℃~+155℃ Operating Temperature:-55℃~+155℃"
+		(property "Description" "Type:Thick Film Resistor Resistance:60.4Ω Tolerance:±1% Power(Watts):500mW Voltage-Supply(Max):400V Temperature Coefficient:±100ppm/℃ Operating Temperature:-55℃~+155℃"
 			(at 134.62 199.39 0)
 			(hide yes)
@@
 			)
 		)
-		(property "Manufacturer Part" "FRC0603F60R4TS"
+		(property "Manufacturer Part" "ERJP06F60R4V"
 			(at 134.62 199.39 0)
 			(hide yes)
@@
 			)
 		)
-		(property "Manufacturer" "FOJAN(富捷)"
+		(property "Manufacturer" "PANASONIC"
 			(at 134.62 199.39 0)
 			(hide yes)
@@
 			)
 		)
-		(property "Supplier Part" "C2933247"
+		(property "Supplier Part" "C3959530"
 			(at 134.62 199.39 0)
 			(hide yes)
@@
 			)
 		)
-		(property "LCSC Part Name" "60.4Ω ±1% 100mW 厚膜电阻"
+		(property "LCSC Part Name" "ERJP06F60R4V"
 			(at 134.62 199.39 0)
 			(hide yes)
